File: PCB/NIOKR.kicad_pcb (KiCad board)
At the start: 2 copper layers, 143.9 x 99.7 mm, 47 parts

Commit message: minimal-updates
Parts:
- added U?: xiao-ble-thruhole, TOTEMlib:xiao-ble-smd-cutout, F.Cu at (228.0, 158.7)
- moved L-PSW1 124.4 mm to (98.2, 194.6), turned to 90 degrees
- moved L-RSW1 95.6 mm to (86.4, 210.8)
- moved L-MCU1 74.3 mm to (119.1, 177.3), turned to 180 degrees
- moved BATGND1 18.6 mm to (90.1, 185.8)
- moved L-D20 17.7 mm to (168.2, 178.1), turned to -9 degrees
- moved L-D13 15.7 mm to (89.7, 161.9), turned to -81 degrees
- moved L-D12 15.6 mm to (70.4, 164.4), turned to -81 degrees
- moved BAT+1 12.9 mm to (89.5, 182.4)
- moved L-D11 5.45 mm to (162.5, 150.6), turned to 0 degrees
- moved L-D7 5.40 mm to (88.3, 152.6), turned to 99 degrees
- moved L-D5 5.30 mm to (162.5, 131.0), turned to 0 degrees
- moved L-D1 5.17 mm to (85.3, 133.2), turned to 99 degrees
- moved L-D6 5.06 mm to (68.8, 155.8), turned to 99 degrees
- moved L-D16 4.35 mm to (142.9, 169.8), turned to 0 degrees
- moved L-D18 4.32 mm to (143.0, 175.0), turned to 0 degrees
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Other:
- board size 143.9 x 99.7 mm -> 324.1 x 141 mm

Commit message: houdini routing
Parts:
- removed BAT+1: +, TOTEMlib:BatteryPad
- removed BATGND1: -, TOTEMlib:BatteryPad
- removed L-MCU1: Nice_Nano_V2, MCU:Nice_Nano_V2
- removed L-RSW1: Reset, TOTEMlib:SKHLLCA010
- removed U?: xiao-ble-thruhole, TOTEMlib:xiao-ble-smd-cutout
- added L-BAT+1: MountingHole_Pad_MP, TOTEMlib:BatteryPad, F.Cu at (121.4, 159.7)
- added L-GND1: MountingHole_Pad_MP, TOTEMlib:BatteryPad, F.Cu at (117.4, 159.8)
- added U1: XIAO-nRF52840-SMD, Seeed Studio XIAO Series Library:XIAO-nRF52840-SMD, F.Cu at (111.5, 183.5)
- L-S0, L-S1, L-S2, L-S3, L-S4, L-S5: footprint Hotswap:Hotswap_Choc_V1V2_neri_klp_saddle_tilted_top -> Hotswap:Hotswap_Choc_V1V2_klp_saddle
- L-S10: footprint Hotswap:Hotswap_Choc_V1V2_klp_saddle_homing -> Hotswap:Hotswap_Choc_V1V2_klp_saddle
- L-S12, L-S13, L-S14, L-S15, L-S16, L-S17: footprint Hotswap:Hotswap_Choc_V1V2_neri_klp_saddle_tilted_bottom -> Hotswap:Hotswap_Choc_V1V2_klp_saddle
- L-S18, L-S19, L-S20: footprint Hotswap:Hotswap_Choc_V1V2_neri_klp_saddle_thumb -> Hotswap:Hotswap_Choc_V1V2_klp_saddle
- moved L-PSW1 14.7 mm to (83.5, 193.4)
Other:
- board size 324.1 x 141 mm -> 149.8 x 103 mm

Commit message: current
Parts:
- added L-BAT+2: +, NII:BatteryPad, F.Cu at (117.6, 173.0)
- added R-BAT+1: +, NII:BatteryPad, F.Cu at (281.2, 148.6)
- added R-BAT+2: +, NII:BatteryPad, F.Cu at (271.2, 173.0)
- added R-D0: Diode, NII:Diode_SOD123, B.Cu at (329.4, 122.4)
- added R-D03: Diode, NII:Diode_SOD123, B.Cu at (272.4, 95.4)
- added R-D1: Diode, NII:Diode_SOD123, B.Cu at (311.1, 119.6)
- added R-D10: Diode, NII:Diode_SOD123, B.Cu at (251.5, 127.3)
- added R-D11: Diode, NII:Diode_SOD123, B.Cu at (233.0, 127.3)
- added R-D12: Diode, NII:Diode_SOD123, B.Cu at (323.6, 159.0)
- added R-D13: Diode, NII:Diode_SOD123, B.Cu at (305.4, 156.1)
- added R-D14: Diode, NII:Diode_SOD123, B.Cu at (288.9, 138.9)
- added R-D15: Diode, NII:Diode_SOD123, B.Cu at (270.5, 132.4)
- added R-D16: Diode, NII:Diode_SOD123, B.Cu at (251.5, 145.8)
- added R-D17: Diode, NII:Diode_SOD123, B.Cu at (233.0, 145.8)
- added R-D18: Diode, NII:Diode_SOD123, B.Cu at (251.5, 170.8)
- added R-D19: Diode, NII:Diode_SOD123, B.Cu at (233.0, 170.8)
- added R-D2: Diode, NII:Diode_SOD123, B.Cu at (292.8, 102.1)
- added R-D20: Diode, NII:Diode_SOD123, B.Cu at (212.6, 173.5)
- added R-D4: Diode, NII:Diode_SOD123, B.Cu at (251.5, 108.8)
- added R-D5: Diode, NII:Diode_SOD123, B.Cu at (233.0, 108.8)
- added R-D6: Diode, NII:Diode_SOD123, B.Cu at (326.5, 140.7)
- added R-D7: Diode, NII:Diode_SOD123, B.Cu at (308.2, 137.8)
- added R-D8: Diode, NII:Diode_SOD123, B.Cu at (290.9, 120.5)
- added R-D9: Diode, NII:Diode_SOD123, B.Cu at (271.4, 113.9)
- added R-GND1: -, NII:BatteryPad, F.Cu at (275.2, 148.6)
- added R-PSW1: Power, NII:MSK12C02, F.Cu at (334.8, 183.7)
- added R-S0: Keyswitch, NII:keyswitch_choc12_gateron_low_profile_hotswap_1u_no_led, F.Cu at (335.7, 127.7)
- added R-S1: Keyswitch, NII:keyswitch_choc12_gateron_low_profile_hotswap_1u_no_led, F.Cu at (317.4, 124.8)
- added R-S10: Keyswitch, NII:keyswitch_choc12_gateron_low_profile_hotswap_1u_no_led, F.Cu at (258.5, 131.5)
- added R-S11: Keyswitch, NII:keyswitch_choc12_gateron_low_profile_hotswap_1u_no_led, F.Cu at (240.0, 131.5)
- added R-S12: Keyswitch, NII:keyswitch_choc12_gateron_low_profile_hotswap_1u_no_led, F.Cu at (329.9, 164.2)
- added R-S13: Keyswitch, NII:keyswitch_choc12_gateron_low_profile_hotswap_1u_no_led, F.Cu at (311.6, 161.3)
- added R-S14: Keyswitch, NII:keyswitch_choc12_gateron_low_profile_hotswap_1u_no_led, F.Cu at (295.5, 143.8)
- added R-S15: Keyswitch, NII:keyswitch_choc12_gateron_low_profile_hotswap_1u_no_led, F.Cu at (277.2, 136.9)
- added R-S16: Keyswitch, NII:keyswitch_choc12_gateron_low_profile_hotswap_1u_no_led, F.Cu at (258.5, 150.0)
- added R-S17: Keyswitch, NII:keyswitch_choc12_gateron_low_profile_hotswap_1u_no_led, F.Cu at (240.0, 150.0)
- added R-S18: Keyswitch, NII:keyswitch_choc12_gateron_low_profile_hotswap_1u_no_led, F.Cu at (258.5, 175.0)
- added R-S19: Keyswitch, NII:keyswitch_choc12_gateron_low_profile_hotswap_1u_no_led, F.Cu at (240.0, 175.0)
- added R-S2: Keyswitch, NII:keyswitch_choc12_gateron_low_profile_hotswap_1u_no_led, F.Cu at (299.3, 107.0)
- added R-S20: Keyswitch, NII:keyswitch_choc12_gateron_low_profile_hotswap_1u_no_led, F.Cu at (220.2, 176.6)
- added R-S3: Keyswitch, NII:keyswitch_choc12_gateron_low_profile_hotswap_1u_no_led, F.Cu at (279.2, 100.0)
- added R-S4: Keyswitch, NII:keyswitch_choc12_gateron_low_profile_hotswap_1u_no_led, F.Cu at (258.5, 113.0)
- added R-S5: Keyswitch, NII:keyswitch_choc12_gateron_low_profile_hotswap_1u_no_led, F.Cu at (240.0, 113.0)
- added R-S6: Keyswitch, NII:keyswitch_choc12_gateron_low_profile_hotswap_1u_no_led, F.Cu at (332.8, 146.0)
- added R-S7: Keyswitch, NII:keyswitch_choc12_gateron_low_profile_hotswap_1u_no_led, F.Cu at (314.5, 143.1)
- added R-S8: Keyswitch, NII:keyswitch_choc12_gateron_low_profile_hotswap_1u_no_led, F.Cu at (297.4, 125.4)
- added R-S9: Keyswitch, NII:keyswitch_choc12_gateron_low_profile_hotswap_1u_no_led, F.Cu at (278.2, 118.5)
- added U2: XIAO-nRF52840-SMD, NII:XIAO-nRF52840-cutout, B.Cu at (284.3, 173.0)
- added mbites1: mousebites 2mm, NII:mousebites_0.6-0.4, F.Cu at (185.0, 124.9)
- added mbites2: mousebites 2mm, NII:mousebites_0.6-0.4, F.Cu at (185.0, 142.9)
- added mbites3: mousebites 2mm, NII:mousebites_0.6-0.4, F.Cu at (230.0, 124.9)
- added mbites4: mousebites 2mm, NII:mousebites_0.6-0.4, F.Cu at (230.0, 142.9)
- L-BAT+1: value MountingHole_Pad_MP -> +; footprint TOTEMlib:BatteryPad -> NII:BatteryPad
- L-D0, L-D1, L-D10, L-D11, L-D12, L-D13, L-D14, L-D15, L-D16, L-D17, L-D18, L-D19, L-D2, L-D20, L-D3, L-D4, L-D5, L-D6, L-D7, L-D8, L-D9: footprint Diode_SMD:D_SOD-123 -> NII:Diode_SOD123
- L-GND1: value MountingHole_Pad_MP -> -; footprint TOTEMlib:BatteryPad -> NII:BatteryPad
- L-PSW1: footprint TOTEMlib:MSK12C02 -> NII:MSK12C02
- L-S0, L-S1, L-S10, L-S11, L-S12, L-S13, L-S14, L-S15, L-S16, L-S17, L-S18, L-S19, L-S2, L-S20, L-S3, L-S4, L-S5, L-S6, L-S7, L-S8, L-S9: footprint Hotswap:Hotswap_Choc_V1V2_klp_saddle -> NII:keyswitch_choc12_gateron_low_profile_hotswap_1u_no_led
- U1: footprint Seeed Studio XIAO Series Library:XIAO-nRF52840-SMD -> NII:XIAO-nRF52840-cutout; moved to B.Cu
- moved L-S12 25.4 mm to (85.1, 164.2)
- moved L-S6 25.1 mm to (82.2, 146.0)
- moved L-GND1 25.1 mm to (139.8, 148.5)
- moved L-D16 24.9 mm to (149.5, 145.8), turned to 90 degrees
- moved L-S0 24.9 mm to (79.3, 127.7)
- moved L-D17 24.6 mm to (168.0, 145.8), turned to 90 degrees
- moved L-S13 24.5 mm to (103.4, 161.3)
- moved L-S7 24.2 mm to (100.5, 143.1)
- moved L-S1 23.9 mm to (97.6, 124.8)
- moved L-D11 23.9 mm to (168.0, 127.3), turned to 90 degrees
- moved L-S14 23.5 mm to (119.5, 143.8)
- moved L-S8 23.1 mm to (117.6, 125.4)
- moved L-D5 22.9 mm to (168.0, 108.8), turned to 90 degrees
- moved L-S2 22.8 mm to (115.7, 107.0)
- moved L-S15 22.5 mm to (137.8, 136.9)
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Connections:
- U1 pad 1: L-COL0 -> L-ROW3
- U1 pad 10: L-ROW1 -> L-COL2
- U1 pad 12: unconnected-(U1-3V3-Pad12) -> L-ROW1
- U1 pad 2: L-COL1 -> L-ROW2
- U1 pad 3: L-COL2 -> L-COL5
- U1 pad 4: L-COL3 -> L-COL4
- U1 pad 5: L-COL4 -> L-COL3
- U1 pad 6: L-COL5 -> unconnected-(U1-P0.05_A5_D5_SCL-Pad6)
- U1 pad 8: L-ROW3 -> L-COL0
- U1 pad 9: L-ROW2 -> L-COL1
Routing:
- net R-ROW3: vias 0 -> 1
- net R-ROW2: vias 0 -> 5
- net R-ROW1: vias 0 -> 5
- net R-ROW0: vias 0 -> 4
- net R-GND: vias 0 -> 1
- net R-COL5: vias 0 -> 1
- net R-COL4: vias 0 -> 1
- net R-COL3: vias 0 -> 1
- net R-COL1: vias 0 -> 2
- net R-COL0: vias 0 -> 1
- net L-ROW3: vias 0 -> 1
- net L-ROW2: vias 0 -> 3
- net L-ROW1: vias 0 -> 6
- net L-ROW0: vias 0 -> 2
- net L-COL4: vias 0 -> 1
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Other:
- board size 149.8 x 103 mm -> 278.7 x 101.2 mm

Commit message: wip v2
Parts:
- L-S0, L-S1, L-S10, L-S11, L-S12, L-S13, L-S14, L-S15, L-S16, L-S17, L-S18, L-S19, L-S2, L-S20, L-S3, L-S4, L-S5, L-S6, L-S7, L-S8, L-S9, R-S0, R-S1, R-S10, R-S11, R-S12, R-S13, R-S14, R-S15, R-S16, R-S17, R-S18, R-S19, R-S2, R-S20, R-S3, R-S4, R-S5, R-S6, R-S7, R-S8, R-S9: footprint NII:keyswitch_choc12_gateron_low_profile_hotswap_1u_no_led -> NII:keyswitch_chocv2
- moved R-D20 19.7 mm to (222.9, 190.3), turned to -166.5 degrees
- moved L-D20 19.1 mm to (187.1, 190.3), turned to -13.5 degrees
- moved R-D19 17.1 mm to (240.9, 186.0), turned to -166.5 degrees
- moved L-D19 15.3 mm to (169.1, 186.0), turned to -13.5 degrees
- moved L-PSW1 14.6 mm to (66.1, 168.3), turned to 0 degrees
- moved R-D17 13.5 mm to (240.5, 157.0), turned to -175.5 degrees
- moved R-D18 13.2 mm to (258.9, 181.7), turned to -166.5 degrees
- moved R-D11 12.8 mm to (239.1, 138.5), turned to -175.5 degrees
- moved R-D16 12.3 mm to (259.0, 155.5), turned to -175.5 degrees
- moved R-D5 12.2 mm to (237.6, 120.1), turned to -175.5 degrees
- moved L-D5 12.1 mm to (172.4, 120.1), turned to 175.5 degrees
- moved R-PSW1 11.9 mm to (343.9, 176.0), turned to 180 degrees
- moved L-D11 11.6 mm to (170.9, 138.5), turned to 175.5 degrees
- moved R-D10 11.5 mm to (257.5, 137.1), turned to -175.5 degrees
- moved L-D17 11.3 mm to (169.5, 157.0), turned to 175.5 degrees
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Connections:
- U1 pad 11: L-ROW0 -> L-COL3
- U1 pad 12: L-ROW1 -> unconnected-(U1-3V3-Pad12)
- U1 pad 3: L-COL5 -> L-ROW1
- U1 pad 4: L-COL4 -> L-ROW0
- U1 pad 5: L-COL3 -> L-COL5
- U1 pad 6: unconnected-(U1-P0.05_A5_D5_SCL-Pad6) -> L-COL4
Routing:
- net R-ROW3: vias 1 -> 0
- net R-ROW2: vias 5 -> 0
- net R-ROW1: vias 5 -> 0
- net R-ROW0: vias 4 -> 0
- net R-GND: vias 1 -> 0
- net R-COL5: vias 1 -> 0
- net R-COL4: vias 1 -> 0
- net R-COL3: vias 1 -> 0
- net R-COL1: vias 2 -> 0
- net R-COL0: vias 1 -> 0
- net L-ROW3: vias 1 -> 0
- net L-ROW2: vias 3 -> 0
- net L-ROW1: vias 6 -> 0
- net L-ROW0: vias 2 -> 0
- net L-COL4: vias 1 -> 0
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Other:
- board size 278.7 x 101.2 mm -> 278.8 x 108.6 mm

Commit message: Pipeline_preparation
Parts:
- added mbites5: mousebites 2mm, NII:mousebites_0.6-0.4, F.Cu at (-54.3, -23.2)
- added mbites6: mousebites 2mm, NII:mousebites_0.6-0.4, F.Cu at (-54.3, -3.16)
- added mbites7: mousebites 2mm, NII:mousebites_0.6-0.4, F.Cu at (-15.7, -23.2)
- added mbites8: mousebites 2mm, NII:mousebites_0.6-0.4, F.Cu at (-15.7, -3.16)
- U1, U2: footprint NII:XIAO-nRF52840-cutout -> NII:XIAO-nRF52840-cutout-plain
- moved L-BAT+1 285.4 mm to (-109.4, -0.75)
- moved L-GND1 285.4 mm to (-103.4, -0.75)
- moved R-D18 285.0 mm to (18.2, 29.0)
- moved R-S18 285.0 mm to (16.6, 22.2)
- moved R-S19 285.0 mm to (-1.38, 26.5)
- moved R-S20 285.0 mm to (-19.4, 30.9)
- moved R-D19 285.0 mm to (0.26, 33.3)
- moved R-D20 285.0 mm to (-17.7, 37.7)
- moved R-BAT+1 284.2 mm to (39.4, -0.75)
- moved R-GND1 284.2 mm to (33.4, -0.75)
- moved L-D18 283.9 mm to (-88.2, 29.0)
- moved L-D20 283.9 mm to (-52.3, 37.7)
- moved L-S18 283.9 mm to (-86.6, 22.2)
- moved L-S19 283.9 mm to (-68.6, 26.5)
- moved L-S20 283.9 mm to (-50.6, 30.9)
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Connections:
- U2 pad 1: R-COL0 -> R-ROW3
- U2 pad 10: R-COL5 -> R-COL2
- U2 pad 11: R-COL4 -> R-COL3
- U2 pad 12: R-COL3 -> unconnected-(U2-3V3-Pad12)
- U2 pad 2: R-COL1 -> R-ROW2
- U2 pad 3: R-COL2 -> R-ROW1
- U2 pad 5: R-ROW1 -> R-COL5
- U2 pad 6: unconnected-(U2-P0.05_A5_D5_SCL-Pad6) -> R-COL4
- U2 pad 8: R-ROW3 -> R-COL0
- U2 pad 9: R-ROW2 -> R-COL1
Other:
- board size 278.8 x 108.6 mm -> 278.8 x 106 mm
- board text added: "L-Front"

Commit message: wip pattern
Parts:
- turned L-D18 to 166.5 degrees
- turned L-D19 to 166.5 degrees
- turned L-D20 to 166.5 degrees
Changed lines of the file:
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@@
 		(placed yes)
 		(layer "B.Cu")
-		(at -70.255065 33.344116 -13.5)
+		(at -70.255065 33.344116 166.5)
 		(descr "Diode, DO-41, SOD81, Horizontal, RM 10mm,")
 		(tags "Diode, DO-41, SOD81, Horizontal, RM 10mm, 1N4007, SB140,")
@@
 		(attr through_hole)
 		(fp_line
-			(start -0.5 0.7)
-			(end -0.5 -0.7)
+			(start 0.4 -0.7)
+			(end -0.5 0)
 			(stroke
 				(width 0.15)
@@
 		)
 		(fp_line
-			(start -0.5 0)
-			(end 0.4 0.7)
+			(start 0.4 0.7)
+			(end 0.4 -0.7)
 			(stroke
 				(width 0.15)
@@
 		)
 		(fp_line
-			(start 0.4 0.7)
-			(end 0.4 -0.7)
+			(start -0.5 0)
+			(end 0.4 0.7)
 			(stroke
 				(width 0.15)
@@
 		)
 		(fp_line
-			(start 0.4 -0.7)
-			(end -0.5 0)
+			(start -0.5 0.7)
+			(end -0.5 -0.7)
 			(stroke
 				(width 0.15)
@@
 		)
 		(pad "1" smd roundrect
-			(at -1.7 0 346.5)
+			(at -1.7 0 166.5)
 			(size 1.8 1.5)
 			(layers "B.Cu" "B.Mask" "B.Paste")
@@
 		)
 		(pad "2" smd roundrect
-			(at 1.7 0 346.5)
+			(at 1.7 0 166.5)
 			(size 1.8 1.5)
 			(layers "B.Cu" "B.Mask" "B.Paste")
@@
 		(placed yes)
 		(layer "B.Cu")
-		(at -52.266222 37.662855 -13.5)
+		(at -52.266222 37.662855 166.5)
 		(descr "Diode, DO-41, SOD81, Horizontal, RM 10mm,")
 		(tags "Diode, DO-41, SOD81, Horizontal, RM 10mm, 1N4007, SB140,")
@@
 		(attr through_hole)
 		(fp_line
-			(start -0.5 0.7)
-			(end -0.5 -0.7)
+			(start 0.4 -0.7)
+			(end -0.5 0)
 			(stroke
 				(width 0.15)
@@
 		)
 		(fp_line
-			(start -0.5 0)
-			(end 0.4 0.7)
+			(start 0.4 0.7)
+			(end 0.4 -0.7)
 			(stroke
 				(width 0.15)
@@
 		)
 		(fp_line
-			(start 0.4 0.7)
-			(end 0.4 -0.7)
+			(start -0.5 0)
+			(end 0.4 0.7)
 			(stroke
 				(width 0.15)
@@
 		)
 		(fp_line
-			(start 0.4 -0.7)
-			(end -0.5 0)
+			(start -0.5 0.7)
+			(end -0.5 -0.7)
 			(stroke
 				(width 0.15)
@@
 		)
 		(pad "1" smd roundrect
-			(at -1.7 0 346.5)
+			(at -1.7 0 166.5)
 			(size 1.8 1.5)
 			(layers "B.Cu" "B.Mask" "B.Paste")
@@
 		)
 		(pad "2" smd roundrect
-			(at 1.7 0 346.5)
+			(at 1.7 0 166.5)
 			(size 1.8 1.5)
 			(layers "B.Cu" "B.Mask" "B.Paste")
@@
 		(placed yes)
 		(layer "B.Cu")
-		(at -88.243911 29.025376 -13.5)
+		(at -88.243911 29.025376 166.5)
 		(descr "Diode, DO-41, SOD81, Horizontal, RM 10mm,")
 		(tags "Diode, DO-41, SOD81, Horizontal, RM 10mm, 1N4007, SB140,")
@@
 		(attr through_hole)
 		(fp_line
-			(start -0.5 0.7)
-			(end -0.5 -0.7)
+			(start 0.4 -0.7)
+			(end -0.5 0)
 			(stroke
 				(width 0.15)
@@
 		)
 		(fp_line
-			(start -0.5 0)
-			(end 0.4 0.7)
+			(start 0.4 0.7)
+			(end 0.4 -0.7)
 			(stroke
 				(width 0.15)
@@
 		)
 		(fp_line
-			(start 0.4 0.7)
-			(end 0.4 -0.7)
+			(start -0.5 0)
+			(end 0.4 0.7)
 			(stroke
 				(width 0.15)
@@
 		)
 		(fp_line
-			(start 0.4 -0.7)
-			(end -0.5 0)
+			(start -0.5 0.7)
+			(end -0.5 -0.7)
 			(stroke
 				(width 0.15)
@@
 		)
 		(pad "1" smd roundrect
-			(at -1.7 0 346.5)
+			(at -1.7 0 166.5)
 			(size 1.8 1.5)
 			(layers "B.Cu" "B.Mask" "B.Paste")
@@
 		)
 		(pad "2" smd roundrect
-			(at 1.7 0 346.5)
+			(at 1.7 0 166.5)
 			(size 1.8 1.5)
 			(layers "B.Cu" "B.Mask" "B.Paste")

Commit message: algo almost done + chocv1
Parts:
- L-S0, L-S1, L-S10, L-S11, L-S12, L-S13, L-S14, L-S15, L-S16, L-S17, L-S18, L-S19, L-S2, L-S20, L-S3, L-S4, L-S5, L-S6, L-S7, L-S8, L-S9, R-S0, R-S1, R-S10, R-S11, R-S12, R-S13, R-S14, R-S15, R-S16, R-S17, R-S18, R-S19, R-S2, R-S20, R-S3, R-S4, R-S5, R-S6, R-S7, R-S8, R-S9: footprint NII:keyswitch_chocv2 -> NII:keyswitch_choc12-topor
- mbites1, mbites2, mbites3, mbites4, mbites5, mbites6, mbites7, mbites8: footprint NII:mousebites_0.6-0.4 -> NII:mousebites_0.6-0.4-topor
- moved mbites8 3.75 mm to (-15.5, 0.59)
- moved mbites6 3.75 mm to (-54.5, 0.59)
- moved mbites4 3.75 mm to (-13.5, 0.59)
- moved mbites2 3.75 mm to (-56.5, 0.58)
- moved mbites1 2.75 mm to (-56.5, -20.4)
- moved mbites5 2.75 mm to (-54.5, -20.4)
- moved mbites7 2.75 mm to (-15.5, -20.4)
- moved mbites3 2.75 mm to (-13.5, -20.4)
- moved R-D03 2.04 mm to (35.3, -43.9)
- moved L-S3 2.00 mm to (-105.2, -50.9)
- moved R-S3 2.00 mm to (35.2, -50.9)
- moved L-S0 2.00 mm to (-163.5, -27.8)
- moved L-S1 2.00 mm to (-145.0, -29.2)
- moved L-D4 2.00 mm to (-86.2, -29.4)
- moved R-D5 2.00 mm to (-2.20, -27.9)
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Other:
- board size 278.8 x 106 mm -> 278.4 x 103 mm
- board text removed: "L-Front"
