File: PCB/NIOKR.kicad_sch (KiCad schematic)
At the start: 94 parts, among them U1 XIAO-nRF52840-SMD, U2 XIAO-nRF52840-SMD

Commit message: algo almost done + chocv1
Parts:
- L-S0, L-S1, L-S10, L-S11, L-S12, L-S13, L-S14, L-S15, L-S16, L-S17, L-S18, L-S19, L-S2, L-S20, L-S3, L-S4, L-S5, L-S6, L-S7, L-S8, L-S9, R-S0, R-S1, R-S10, R-S11, R-S12, R-S13, R-S14, R-S15, R-S16, R-S17, R-S18, R-S19, R-S2, R-S20, R-S3, R-S4, R-S5, R-S6, R-S7, R-S8, R-S9: footprint NII:keyswitch_chocv2_topor -> NII:keyswitch_choc12-topor
Changed lines of the file:
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@@
 			)
 		)
-		(property "Footprint" "NII:keyswitch_chocv2_topor"
+		(property "Footprint" "NII:keyswitch_choc12-topor"
 			(at 344.17 128.27 0)
 			(effects
@@
 			)
 		)
-		(property "Footprint" "NII:keyswitch_chocv2_topor"
+		(property "Footprint" "NII:keyswitch_choc12-topor"
 			(at 129.54 129.54 0)
 			(effects
@@
 			)
 		)
-		(property "Footprint" "NII:keyswitch_chocv2_topor"
+		(property "Footprint" "NII:keyswitch_choc12-topor"
 			(at 91.44 78.74 0)
 			(effects
@@
 			)
 		)
-		(property "Footprint" "NII:keyswitch_chocv2_topor"
+		(property "Footprint" "NII:keyswitch_choc12-topor"
 			(at 280.67 102.87 0)
 			(effects
@@
 			)
 		)
-		(property "Footprint" "NII:keyswitch_chocv2_topor"
+		(property "Footprint" "NII:keyswitch_choc12-topor"
 			(at 116.84 104.14 0)
 			(effects
@@
 			)
 		)
-		(property "Footprint" "NII:keyswitch_chocv2_topor"
+		(property "Footprint" "NII:keyswitch_choc12-topor"
 			(at 104.14 129.54 0)
 			(effects
@@
 			)
 		)
-		(property "Footprint" "NII:keyswitch_chocv2_topor"
+		(property "Footprint" "NII:keyswitch_choc12-topor"
 			(at 129.54 154.94 0)
 			(effects
@@
 			)
 		)
-		(property "Footprint" "NII:keyswitch_chocv2_topor"
+		(property "Footprint" "NII:keyswitch_choc12-topor"
 			(at 318.77 102.87 0)
 			(effects
@@
 			)
 		)
-		(property "Footprint" "NII:keyswitch_chocv2_topor"
+		(property "Footprint" "NII:keyswitch_choc12-topor"
 			(at 344.17 77.47 0)
 			(effects
@@
 			)
 		)
-		(property "Footprint" "NII:keyswitch_chocv2_topor"
+		(property "Footprint" "NII:keyswitch_choc12-topor"
 			(at 116.84 78.74 0)
 			(effects
@@
 			)
 		)
-		(property "Footprint" "NII:keyswitch_chocv2_topor"
+		(property "Footprint" "NII:keyswitch_choc12-topor"
 			(at 280.67 77.47 0)
 			(effects
@@
 			)
 		)
-		(property "Footprint" "NII:keyswitch_chocv2_topor"
+		(property "Footprint" "NII:keyswitch_choc12-topor"
 			(at 280.67 153.67 0)
 			(effects
@@
 			)
 		)
-		(property "Footprint" "NII:keyswitch_chocv2_topor"
+		(property "Footprint" "NII:keyswitch_choc12-topor"
 			(at 116.84 129.54 0)
 			(effects
@@
 			)
 		)
-		(property "Footprint" "NII:keyswitch_chocv2_topor"
+		(property "Footprint" "NII:keyswitch_choc12-topor"
 			(at 104.14 104.14 0)
 			(effects
@@
 			)
 		)
-		(property "Footprint" "NII:keyswitch_chocv2_topor"
+		(property "Footprint" "NII:keyswitch_choc12-topor"
 			(at 306.07 77.47 0)
 			(effects
@@
 			)
 		)
-		(property "Footprint" "NII:keyswitch_chocv2_topor"
+		(property "Footprint" "NII:keyswitch_choc12-topor"
 			(at 293.37 77.47 0)
 			(effects
@@
 			)
 		)
-		(property "Footprint" "NII:keyswitch_chocv2_topor"
+		(property "Footprint" "NII:keyswitch_choc12-topor"
 			(at 344.17 102.87 0)
 			(effects
@@
 			)
 		)
-		(property "Footprint" "NII:keyswitch_chocv2_topor"
+		(property "Footprint" "NII:keyswitch_choc12-topor"
 			(at 318.77 77.47 0)
 			(effects
@@
 			)
 		)
-		(property "Footprint" "NII:keyswitch_chocv2_topor"
+		(property "Footprint" "NII:keyswitch_choc12-topor"
 			(at 293.37 102.87 0)
 			(effects
@@
 			)
 		)
-		(property "Footprint" "NII:keyswitch_chocv2_topor"
+		(property "Footprint" "NII:keyswitch_choc12-topor"
 			(at 91.44 104.14 0)
 			(effects
@@
 			)
 		)
-		(property "Footprint" "NII:keyswitch_chocv2_topor"
+		(property "Footprint" "NII:keyswitch_choc12-topor"
 			(at 293.37 153.67 0)
 			(effects
@@
 			)
 		)
-		(property "Footprint" "NII:keyswitch_chocv2_topor"
+		(property "Footprint" "NII:keyswitch_choc12-topor"
 			(at 78.74 129.54 0)
 			(effects
@@
 			)
 		)
-		(property "Footprint" "NII:keyswitch_chocv2_topor"
+		(property "Footprint" "NII:keyswitch_choc12-topor"
 			(at 78.74 78.74 0)
 			(effects
@@
 			)
 		)
-		(property "Footprint" "NII:keyswitch_chocv2_topor"
+		(property "Footprint" "NII:keyswitch_choc12-topor"
 			(at 280.67 128.27 0)
 			(effects
@@
 			)
 		)
-		(property "Footprint" "NII:keyswitch_chocv2_topor"
+		(property "Footprint" "NII:keyswitch_choc12-topor"
 			(at 331.47 77.47 0)
 			(effects
@@
 			)
 		)
-		(property "Footprint" "NII:keyswitch_chocv2_topor"
+		(property "Footprint" "NII:keyswitch_choc12-topor"
 			(at 116.84 154.94 0)
 			(effects
@@
 			)
 		)
-		(property "Footprint" "NII:keyswitch_chocv2_topor"
+		(property "Footprint" "NII:keyswitch_choc12-topor"
 			(at 306.07 153.67 0)
 			(effects
@@
 			)
 		)
-		(property "Footprint" "NII:keyswitch_chocv2_topor"
+		(property "Footprint" "NII:keyswitch_choc12-topor"
 			(at 318.77 128.27 0)
 			(effects
@@
 			)
 		)
-		(property "Footprint" "NII:keyswitch_chocv2_topor"
+		(property "Footprint" "NII:keyswitch_choc12-topor"
 			(at 306.07 102.87 0)
 			(effects
@@
 			)
 		)
-		(property "Footprint" "NII:keyswitch_chocv2_topor"
+		(property "Footprint" "NII:keyswitch_choc12-topor"
 			(at 293.37 128.27 0)
 			(effects
@@
 			)
 		)
-		(property "Footprint" "NII:keyswitch_chocv2_topor"
+		(property "Footprint" "NII:keyswitch_choc12-topor"
 			(at 331.47 102.87 0)
 			(effects
@@
 			)
 		)
-		(property "Footprint" "NII:keyswitch_chocv2_topor"
+		(property "Footprint" "NII:keyswitch_choc12-topor"
 			(at 129.54 104.14 0)
 			(effects
@@
 			)
 		)
-		(property "Footprint" "NII:keyswitch_chocv2_topor"
+		(property "Footprint" "NII:keyswitch_choc12-topor"
 			(at 66.04 129.54 0)
 			(effects
@@
 			)
 		)
-		(property "Footprint" "NII:keyswitch_chocv2_topor"
+		(property "Footprint" "NII:keyswitch_choc12-topor"
 			(at 66.04 78.74 0)
 			(effects
@@
 			)
 		)
-		(property "Footprint" "NII:keyswitch_chocv2_topor"
+		(property "Footprint" "NII:keyswitch_choc12-topor"
 			(at 306.07 128.27 0)
 			(effects
@@
 			)
 		)
-		(property "Footprint" "NII:keyswitch_chocv2_topor"
+		(property "Footprint" "NII:keyswitch_choc12-topor"
 			(at 66.04 104.14 0)
 			(effects
@@
 			)
 		)
-		(property "Footprint" "NII:keyswitch_chocv2_topor"
+		(property "Footprint" "NII:keyswitch_choc12-topor"
 			(at 91.44 129.54 0)
 			(effects
@@
 			)
 		)
-		(property "Footprint" "NII:keyswitch_chocv2_topor"
+		(property "Footprint" "NII:keyswitch_choc12-topor"
 			(at 331.47 128.27 0)
 			(effects
@@
 			)
 		)
-		(property "Footprint" "NII:keyswitch_chocv2_topor"
+		(property "Footprint" "NII:keyswitch_choc12-topor"
 			(at 129.54 78.74 0)
 			(effects
@@
 			)
 		)
-		(property "Footprint" "NII:keyswitch_chocv2_topor"
+		(property "Footprint" "NII:keyswitch_choc12-topor"
 			(at 104.14 154.94 0)
 			(effects
@@
 			)
 		)
-		(property "Footprint" "NII:keyswitch_chocv2_topor"
+		(property "Footprint" "NII:keyswitch_choc12-topor"
 			(at 104.14 78.74 0)
 			(effects
@@
 			)
 		)
-		(property "Footprint" "NII:keyswitch_chocv2_topor"
+		(property "Footprint" "NII:keyswitch_choc12-topor"
 			(at 78.74 104.14 0)
 			(effects

Commit message: latest
Parts:
- L-S0, L-S1, L-S10, L-S11, L-S12, L-S13, L-S14, L-S15, L-S16, L-S17, L-S18, L-S19, L-S2, L-S20, L-S3, L-S4, L-S5, L-S6, L-S7, L-S8, L-S9, R-S0, R-S1, R-S10, R-S11, R-S12, R-S13, R-S14, R-S15, R-S16, R-S17, R-S18, R-S19, R-S2, R-S20, R-S3, R-S4, R-S5, R-S6, R-S7, R-S8, R-S9: footprint NII:keyswitch_choc12-topor -> NII:keyswitch_choc12
Changed lines of the file:
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@@
 			)
 		)
-		(property "Footprint" "NII:keyswitch_choc12-topor"
+		(property "Footprint" "NII:keyswitch_choc12"
 			(at 344.17 128.27 0)
 			(effects
@@
 			)
 		)
-		(property "Footprint" "NII:keyswitch_choc12-topor"
+		(property "Footprint" "NII:keyswitch_choc12"
 			(at 129.54 129.54 0)
 			(effects
@@
 			)
 		)
-		(property "Footprint" "NII:keyswitch_choc12-topor"
+		(property "Footprint" "NII:keyswitch_choc12"
 			(at 91.44 78.74 0)
 			(effects
@@
 			)
 		)
-		(property "Footprint" "NII:keyswitch_choc12-topor"
+		(property "Footprint" "NII:keyswitch_choc12"
 			(at 280.67 102.87 0)
 			(effects
@@
 			)
 		)
-		(property "Footprint" "NII:keyswitch_choc12-topor"
+		(property "Footprint" "NII:keyswitch_choc12"
 			(at 116.84 104.14 0)
 			(effects
@@
 			)
 		)
-		(property "Footprint" "NII:keyswitch_choc12-topor"
+		(property "Footprint" "NII:keyswitch_choc12"
 			(at 104.14 129.54 0)
 			(effects
@@
 			)
 		)
-		(property "Footprint" "NII:keyswitch_choc12-topor"
+		(property "Footprint" "NII:keyswitch_choc12"
 			(at 129.54 154.94 0)
 			(effects
@@
 			)
 		)
-		(property "Footprint" "NII:keyswitch_choc12-topor"
+		(property "Footprint" "NII:keyswitch_choc12"
 			(at 318.77 102.87 0)
 			(effects
@@
 			)
 		)
-		(property "Footprint" "NII:keyswitch_choc12-topor"
+		(property "Footprint" "NII:keyswitch_choc12"
 			(at 344.17 77.47 0)
 			(effects
@@
 			)
 		)
-		(property "Footprint" "NII:keyswitch_choc12-topor"
+		(property "Footprint" "NII:keyswitch_choc12"
 			(at 116.84 78.74 0)
 			(effects
@@
 			)
 		)
-		(property "Footprint" "NII:keyswitch_choc12-topor"
+		(property "Footprint" "NII:keyswitch_choc12"
 			(at 280.67 77.47 0)
 			(effects
@@
 			)
 		)
-		(property "Footprint" "NII:keyswitch_choc12-topor"
+		(property "Footprint" "NII:keyswitch_choc12"
 			(at 280.67 153.67 0)
 			(effects
@@
 			)
 		)
-		(property "Footprint" "NII:keyswitch_choc12-topor"
+		(property "Footprint" "NII:keyswitch_choc12"
 			(at 116.84 129.54 0)
 			(effects
@@
 			)
 		)
-		(property "Footprint" "NII:keyswitch_choc12-topor"
+		(property "Footprint" "NII:keyswitch_choc12"
 			(at 104.14 104.14 0)
 			(effects
@@
 			)
 		)
-		(property "Footprint" "NII:keyswitch_choc12-topor"
+		(property "Footprint" "NII:keyswitch_choc12"
 			(at 306.07 77.47 0)
 			(effects
@@
 			)
 		)
-		(property "Footprint" "NII:keyswitch_choc12-topor"
+		(property "Footprint" "NII:keyswitch_choc12"
 			(at 293.37 77.47 0)
 			(effects
@@
 			)
 		)
-		(property "Footprint" "NII:keyswitch_choc12-topor"
+		(property "Footprint" "NII:keyswitch_choc12"
 			(at 344.17 102.87 0)
 			(effects
@@
 			)
 		)
-		(property "Footprint" "NII:keyswitch_choc12-topor"
+		(property "Footprint" "NII:keyswitch_choc12"
 			(at 318.77 77.47 0)
 			(effects
@@
 			)
 		)
-		(property "Footprint" "NII:keyswitch_choc12-topor"
+		(property "Footprint" "NII:keyswitch_choc12"
 			(at 293.37 102.87 0)
 			(effects
@@
 			)
 		)
-		(property "Footprint" "NII:keyswitch_choc12-topor"
+		(property "Footprint" "NII:keyswitch_choc12"
 			(at 91.44 104.14 0)
 			(effects
@@
 			)
 		)
-		(property "Footprint" "NII:keyswitch_choc12-topor"
+		(property "Footprint" "NII:keyswitch_choc12"
 			(at 293.37 153.67 0)
 			(effects
@@
 			)
 		)
-		(property "Footprint" "NII:keyswitch_choc12-topor"
+		(property "Footprint" "NII:keyswitch_choc12"
 			(at 78.74 129.54 0)
 			(effects
@@
 			)
 		)
-		(property "Footprint" "NII:keyswitch_choc12-topor"
+		(property "Footprint" "NII:keyswitch_choc12"
 			(at 78.74 78.74 0)
 			(effects
@@
 			)
 		)
-		(property "Footprint" "NII:keyswitch_choc12-topor"
+		(property "Footprint" "NII:keyswitch_choc12"
 			(at 280.67 128.27 0)
 			(effects
@@
 			)
 		)
-		(property "Footprint" "NII:keyswitch_choc12-topor"
+		(property "Footprint" "NII:keyswitch_choc12"
 			(at 331.47 77.47 0)
 			(effects
@@
 			)
 		)
-		(property "Footprint" "NII:keyswitch_choc12-topor"
+		(property "Footprint" "NII:keyswitch_choc12"
 			(at 116.84 154.94 0)
 			(effects
@@
 			)
 		)
-		(property "Footprint" "NII:keyswitch_choc12-topor"
+		(property "Footprint" "NII:keyswitch_choc12"
 			(at 306.07 153.67 0)
 			(effects
@@
 			)
 		)
-		(property "Footprint" "NII:keyswitch_choc12-topor"
+		(property "Footprint" "NII:keyswitch_choc12"
 			(at 318.77 128.27 0)
 			(effects
@@
 			)
 		)
-		(property "Footprint" "NII:keyswitch_choc12-topor"
+		(property "Footprint" "NII:keyswitch_choc12"
 			(at 306.07 102.87 0)
 			(effects
@@
 			)
 		)
-		(property "Footprint" "NII:keyswitch_choc12-topor"
+		(property "Footprint" "NII:keyswitch_choc12"
 			(at 293.37 128.27 0)
 			(effects
@@
 			)
 		)
-		(property "Footprint" "NII:keyswitch_choc12-topor"
+		(property "Footprint" "NII:keyswitch_choc12"
 			(at 331.47 102.87 0)
 			(effects
@@
 			)
 		)
-		(property "Footprint" "NII:keyswitch_choc12-topor"
+		(property "Footprint" "NII:keyswitch_choc12"
 			(at 129.54 104.14 0)
 			(effects
@@
 			)
 		)
-		(property "Footprint" "NII:keyswitch_choc12-topor"
+		(property "Footprint" "NII:keyswitch_choc12"
 			(at 66.04 129.54 0)
 			(effects
@@
 			)
 		)
-		(property "Footprint" "NII:keyswitch_choc12-topor"
+		(property "Footprint" "NII:keyswitch_choc12"
 			(at 66.04 78.74 0)
 			(effects
@@
 			)
 		)
-		(property "Footprint" "NII:keyswitch_choc12-topor"
+		(property "Footprint" "NII:keyswitch_choc12"
 			(at 306.07 128.27 0)
 			(effects
@@
 			)
 		)
-		(property "Footprint" "NII:keyswitch_choc12-topor"
+		(property "Footprint" "NII:keyswitch_choc12"
 			(at 66.04 104.14 0)
 			(effects
@@
 			)
 		)
-		(property "Footprint" "NII:keyswitch_choc12-topor"
+		(property "Footprint" "NII:keyswitch_choc12"
 			(at 91.44 129.54 0)
 			(effects
@@
 			)
 		)
-		(property "Footprint" "NII:keyswitch_choc12-topor"
+		(property "Footprint" "NII:keyswitch_choc12"
 			(at 331.47 128.27 0)
 			(effects
@@
 			)
 		)
-		(property "Footprint" "NII:keyswitch_choc12-topor"
+		(property "Footprint" "NII:keyswitch_choc12"
 			(at 129.54 78.74 0)
 			(effects
@@
 			)
 		)
-		(property "Footprint" "NII:keyswitch_choc12-topor"
+		(property "Footprint" "NII:keyswitch_choc12"
 			(at 104.14 154.94 0)
 			(effects
@@
 			)
 		)
-		(property "Footprint" "NII:keyswitch_choc12-topor"
+		(property "Footprint" "NII:keyswitch_choc12"
 			(at 104.14 78.74 0)
 			(effects
@@
 			)
 		)
-		(property "Footprint" "NII:keyswitch_choc12-topor"
+		(property "Footprint" "NII:keyswitch_choc12"
 			(at 78.74 104.14 0)
 			(effects
